File: pcb/FSK-66-20-C.kicad_pcb (KiCad board)
At the start: 2 copper layers, 273.3 x 91.2 mm, 174 parts, among them J1 DX07S016JA3, J2 2x3_F, SW1 SW_Push, SW10 SW_Push, SW11 SW_Push, SW12 SW_Push, SW13 SW_Push, SW14 SW_Push, SW15 SW_Push, SW16 SW_Push, SW17 SW_Push, SW18 SW_Push, SW19 SW_Push, SW2 SW_Push, SW20 SW_Push, SW21 SW_Push, SW22 SW_Push, SW23 SW_Push, SW24 SW_Push, SW25 SW_Push, SW26 SW_Push, SW27 SW_Push, SW28 SW_Push, SW29 SW_Push, SW3 SW_Push, SW30 SW_Push, SW31 SW_Push, SW32 SW_Push, SW33 SW_Push, SW34 SW_Push, SW35 SW_Push, SW36 SW_Push, SW37 SW_Push, SW38 SW_Push, SW39 SW_Push, SW4 SW_Push, SW40 SW_Push, SW41 SW_Push, SW42 SW_Push, SW43 SW_Push, SW44 SW_Push, SW45 SW_Push, SW46 SW_Push, SW47 SW_Push, SW48 SW_Push, SW49 SW_Push, SW5 SW_Push, SW50 SW_Push, SW51 SW_Push, SW52 SW_Push, SW53 SW_Push, SW54 SW_Push, SW55 SW_Push, SW56 SW_Push, SW57 SW_Push, SW58 SW_Push, SW59 SW_Push, SW6 SW_Push, SW60 SW_Push, SW61 SW_Push, SW62 SW_Push, SW63 SW_Push, SW64 SW_Push, SW65 SW_Push, SW66 SW_Push, SW67 SW_Push, SW7 SW_Push, SW8 SW_Push, SW9 SW_Push, U1 ATmega32U4-AU, Y1 16MHz

Commit message: [change]change side holes to no-plated
Parts:
- removed the HOLE at (363.2, 133.3)
- removed the HOLE at (90.2, 133.3)
Other:
- outline, holes or cut-outs redrawn

Commit message: [change]change artwork
Parts:
- removed REF** (x10): MountingHole_2.2mm_M2, MountingHole:MountingHole_2.2mm_M2
- HOLE (x3): footprint hole:PKRH -> lib:PKRH
- SW1, SW10, SW11, SW12, SW13, SW14, SW16, SW17, SW18, SW19, SW2, SW20, SW21, SW22, SW23, SW24, SW25, SW26, SW27, SW3, SW30, SW31, SW32, SW33, SW34, SW35, SW36, SW37, SW38, SW39, SW4, SW40, SW43, SW44, SW45, SW46, SW47, SW48, SW49, SW5, SW50, SW51, SW53, SW54, SW55, SW56, SW57, SW58, SW6, SW62, SW63, SW64, SW65, SW66, SW7, SW8, SW9: footprint keyboard_toms:CherryMX_Choc_V2_1u -> lib:CherryMX_Choc_V2_1u
- SW15, SW28, SW60: footprint keyboard_toms:CherryMX_Choc_V2_1u -> lib:CherryMX_Choc_V2_15u
- SW29, SW52: footprint keyboard_toms:CherryMX_Choc_V2_1u -> lib:CherryMX_Choc_V2_175u
- SW41, SW42, SW59, SW61: footprint keyboard_toms:CherryMX_Choc_V2_1u -> lib:CherryMX_Choc_V2_225u
- moved HOLE 140.1 mm to (145.2, 185.6)
- moved D61 57.6 mm to (149.7, 191.9)
- moved C5 47.5 mm to (90.2, 156.0)
- moved C2 47.5 mm to (90.2, 148.4)
- moved C3 47.5 mm to (90.2, 152.2)
- moved D66 46.9 mm to (60.8, 192.3)
- moved SW67 46.6 mm to (58.3, 146.9)
- moved D65 46.5 mm to (79.1, 192.3)
- moved R2 46.4 mm to (58.3, 113.6)
- moved SW66 46.4 mm to (60.2, 186.2)
- moved HOLE 46.1 mm to (75.6, 129.8)
- moved SW54 45.9 mm to (60.2, 167.2)
- moved SW65 45.7 mm to (79.2, 186.2)
- moved D41 45.5 mm to (71.0, 154.2)
- moved SW53 45.3 mm to (79.2, 167.2)
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Connections:
- J1 pad A8: Net-(J1-PadA8) -> unconnected-(J1-PadA8)
- J1 pad B8: Net-(J1-PadB8) -> unconnected-(J1-PadB8)
- U1 pad 22: Net-(U1-Pad22) -> unconnected-(U1-Pad22)
- U1 pad 26: Net-(U1-Pad26) -> unconnected-(U1-Pad26)
- U1 pad 32: Net-(U1-Pad32) -> unconnected-(U1-Pad32)
- U1 pad 40: Net-(U1-Pad40) -> unconnected-(U1-Pad40)
- U1 pad 41: Net-(U1-Pad41) -> unconnected-(U1-Pad41)
- U1 pad 8: Net-(U1-Pad8) -> unconnected-(U1-Pad8)
Routing:
- net /COL12: track 404.8 -> 269.1 mm, vias 2 -> 4
- net /D3: track 435.6 -> 313.6 mm
- net /D0: track 447.7 -> 342.6 mm, vias 7 -> 4
- net /RESET: track 228.6 -> 168.9 mm, vias 4 -> 6
- net /D2: track 363.8 -> 314.8 mm, vias 6 -> 8
- net VCC: track 231.5 -> 186.8 mm, vias 6 -> 5
- net +5V: track 265.1 -> 221.5 mm, vias 8 -> 6
- net /COL9: track 239.2 -> 204.6 mm, vias 2 -> 0
- net /A2: track 190.8 -> 164.4 mm
- net /COL11: track 274.6 -> 297.8 mm, vias 2 -> 1
- net /COL10: track 248.7 -> 269.6 mm, vias 3 -> 1
- net /A1: track 205.1 -> 184.8 mm, vias 3 -> 2
- net /A0: track 223.1 -> 204.2 mm, vias 2 -> 3
- net /D4: track 310.8 -> 329.4 mm, vias 8 -> 3
- net Net-(D61-Pad2): track 13.0 -> 30.7 mm, vias 0 -> 1
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Other:
- board size 273.3 x 91.2 mm -> 285 x 94.6 mm
- net class Default removed

Commit message: [change]update artwork for board drill
Parts:
- moved HOLE 234.8 mm to (75.6, 129.8)
- moved HOLE 234.3 mm to (309.9, 129.5)
- moved HOLE 0.27 mm to (207.4, 148.6)
Routing:
- net GNDPWR: vias 339 -> 337
Other:
- outline, holes or cut-outs redrawn
Changed lines of the file:
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@@
     (pad_to_mask_clearance 0)
     (pcbplotparams
-      (layerselection 0x00010ec_ffffffff)
+      (layerselection 0x00010fc_ffffffff)
       (plot_on_all_layers_selection 0x0000000_00000000)
       (disableapertmacros false)
-      (usegerberextensions false)
+      (usegerberextensions true)
       (usegerberattributes false)
       (usegerberadvancedattributes true)
-      (creategerberjobfile true)
+      (creategerberjobfile false)
       (dashed_line_dash_ratio 12.000000)
       (dashed_line_gap_ratio 3.000000)
@@
       (drillshape 0)
       (scaleselection 1)
-      (outputdirectory "output/FSK-66-20-C/")
+      (outputdirectory "output/")
     )
   )
@@
     (solder_mask_margin 0.1)
     (attr smd)
-    (fp_text reference "U1" (at -6.35 -5.9 180) (layer "F.SilkS")
+    (fp_text reference "U1" (at -6.35 -5.9) (layer "F.SilkS")
         (effects (font (size 1 1) (thickness 0.15)))
     )
-    (fp_text value "ATmega32U4-AU" (at 12.7 6.8 180) (layer "F.SilkS") hide
+    (fp_text value "ATmega32U4-AU" (at 12.7 6.8) (layer "F.SilkS") hide
         (effects (font (size 1.4 1.4) (thickness 0.05)))
     )
@@
   )
   (footprint "lib:PKRH" (layer "F.Cu")
-    (at 310.45 129.7638)
+    (at 75.6 129.7638)
     (attr exclude_from_pos_files exclude_from_bom)
     (fp_text reference "HOLE" (at 0.1753 5.7861) (layer "F.SilkS") hide
@@
   )
   (footprint "lib:PKRH" (layer "F.Cu")
-    (at 207.45 148.8638)
+    (at 207.45 148.59)
     (attr exclude_from_pos_files exclude_from_bom)
     (fp_text reference "HOLE" (at 0.1753 5.7861) (layer "F.SilkS") hide
@@
   )
   (footprint "hole:PKRHC" (layer "F.Cu")
-    (at 75.6 129.7638)
+    (at 309.88 129.54)
     (attr exclude_from_pos_files exclude_from_bom)
     (fp_text reference "HOLE" (at 0 5.08) (layer "F.SilkS") hide
@@
   (gr_line (start 61.15 191.995) (end 48.45 191.995)
     (stroke (width 0.1) (type solid)) (layer "Cmts.User"))
-  (gr_line (start 50.65 158.903799) (end 50.65 195.4638)
+  (gr_line (start 50.65 159.538799) (end 50.65 194.1938)
     (stroke (width 0.1) (type solid)) (layer "Edge.Cuts"))
   (gr_arc (start 333.155399 158.903799) (mid 331.885401 157.633799) (end 333.1554 156.363801)
     (stroke (width 0.1) (type solid)) (layer "Edge.Cuts"))
-  (gr_line (start 333.1554 156.363801) (end 335.6446 156.3638)
+  (gr_line (start 333.1554 156.363801) (end 335.009662 156.3638)
     (stroke (width 0.1) (type solid)) (layer "Edge.Cuts"))
-  (gr_line (start 333.155399 158.903799) (end 335.6446 158.9038)
+  (gr_line (start 333.155399 158.903799) (end 335.009694 158.9038)
     (stroke (width 0.1) (type solid)) (layer "Edge.Cuts"))
-  (gr_line (start 335.6446 158.9038) (end 335.65 195.4638)
+  (gr_line (start 335.644694 159.538706) (end 335.649812 194.193612)
     (stroke (width 0.1) (type solid)) (layer "Edge.Cuts"))
-  (gr_line (start 335.65 195.4638) (end 50.65 195.4638)
+  (gr_line (start 334.379812 195.4638) (end 51.92 195.4638)
     (stroke (width 0.1) (type solid)) (layer "Edge.Cuts"))
-  (gr_line (start 53.139201 156.3638) (end 50.65 156.363799)
+  (gr_arc (start 335.649812 194.193612) (mid 335.277904 195.091759) (end 334.379812 195.4638)
+    (stroke (width 0.1) (type default)) (layer "Edge.Cuts"))
+  (gr_line (start 53.139201 156.3638) (end 51.285 156.363799)
     (stroke (width 0.1) (type solid)) (layer "Edge.Cuts"))
-  (gr_line (start 335.6446 156.3638) (end 335.65 100.8638)
+  (gr_arc (start 51.285 156.363799) (mid 50.835987 156.177812) (end 50.65 155.728799)
+    (stroke (width 0.1) (type default)) (layer "Edge.Cuts"))
+  (gr_line (start 335.644662 155.728862) (end 335.649876 102.133924)
     (stroke (width 0.1) (type solid)) (layer "Edge.Cuts"))
-  (gr_line (start 53.1392 158.903798) (end 50.65 158.903799)
+  (gr_arc (start 335.009694 158.9038) (mid 335.458674 159.089754) (end 335.644694 159.538706)
+    (stroke (width 0.1) (type default)) (layer "Edge.Cuts"))
+  (gr_arc (start 51.92 195.4638) (mid 51.021974 195.091826) (end 50.65 194.1938)
+    (stroke (width 0.1) (type default)) (layer "Edge.Cuts"))
+  (gr_arc (start 335.644662 155.728862) (mid 335.458653 156.177835) (end 335.009662 156.3638)
+    (stroke (width 0.1) (type default)) (layer "Edge.Cuts"))
+  (gr_arc (start 334.379876 100.8638) (mid 335.277961 101.23581) (end 335.649876 102.133924)
+    (stroke (width 0.1) (type default)) (layer "Edge.Cuts"))
+  (gr_line (start 53.1392 158.903798) (end 51.285 158.903799)
     (stroke (width 0.1) (type solid)) (layer "Edge.Cuts"))
   (gr_arc (start 53.139201 156.3638) (mid 54.4092 157.6338) (end 53.1392 158.903798)
     (stroke (width 0.1) (type solid)) (layer "Edge.Cuts"))
-  (gr_line (start 335.65 100.8638) (end 50.65 100.8638)
+  (gr_line (start 334.379876 100.8638) (end 51.92 100.8638)
     (stroke (width 0.1) (type solid)) (layer "Edge.Cuts"))
-  (gr_line (start 50.65 100.8638) (end 50.65 156.363799)
+  (gr_arc (start 50.65 102.1338) (mid 51.021974 101.235774) (end 51.92 100.8638)
+    (stroke (width 0.1) (type default)) (layer "Edge.Cuts"))
+  (gr_arc (start 50.65 159.538799) (mid 50.835988 159.089787) (end 51.285 158.903799)
+    (stroke (width 0.1) (type default)) (layer "Edge.Cuts"))
+  (gr_line (start 50.65 102.1338) (end 50.65 155.728799)
     (stroke (width 0.1) (type solid)) (layer "Edge.Cuts"))
   (gr_text "." (at 198.294 181.327) (layer "F.SilkS")
@@
     (effects (font (size 1 1) (thickness 0.15)))
   )
-  (gr_text "." (at 194.865 174.85) (layer "F.SilkS")
+  (gr_text "." (at 191.643 174.752) (layer "F.SilkS")
     (effects (font (size 1 1) (thickness 0.15)))
   )
@@
   (via (at 80.9 142.2738) (size 0.8) (drill 0.4) (layers "F.Cu" "B.Cu") (free) (net 2))
   (via (at 78.36 134.6538) (size 0.8) (drill 0.4) (layers "F.Cu" "B.Cu") (free) (net 2))
-  (via (at 309.5 125.7638) (size 0.8) (drill 0.4) (layers "F.Cu" "B.Cu") (free) (net 2))
   (via (at 135.51 161.3238) (size 0.8) (drill 0.4) (layers "F.Cu" "B.Cu") (free) (net 2))
   (via (at 115.19 158.7838) (size 0.8) (drill 0.4) (layers "F.Cu" "B.Cu") (free) (net 2))
@@
   (via (at 252.35 120.6838) (size 0.8) (drill 0.4) (layers "F.Cu" "B.Cu") (free) (net 2))
   (via (at 207.9 144.8138) (size 0.8) (drill 0.4) (layers "F.Cu" "B.Cu") (free) (net 2))
-  (via (at 309.5 132.1138) (size 0.8) (drill 0.4) (layers "F.Cu" "B.Cu") (free) (net 2))
   (via (at 157.227 160.9428) (size 0.8) (drill 0.4) (layers "F.Cu" "B.Cu") (free) (net 2))
   (via (at 65.66 181.6438) (size 0.8) (drill 0.4) (layers "F.Cu" "B.Cu") (free) (net 2))
@@
     (polygon
       (pts
+        (xy 60.072 152.0528)
+        (xy 60.072 150.2748)
+        (xy 61.469 150.2748)
+        (xy 61.469 149.7668)
+        (xy 59.564 149.7668)
+        (xy 59.564 152.0528)
+      )
+    )
+  )
+  (zone (net 0) (net_name "") (layer "F.Cu") (hatch edge 0.5)
+    (connect_pads (clearance 0))
+    (min_thickness 0.25) (filled_areas_thickness no)
+    (keepout (tracks allowed) (vias allowed) (pads allowed) (copperpour not_allowed) (footprints allowed))
+    (fill (thermal_gap 0.5) (thermal_bridge_width 0.5))
+    (polygon
+      (pts
         (xy 91.314 156.3708)
         (xy 91.314 156.8788)
@@
     (polygon
       (pts
+        (xy 154.432 189.738)
+        (xy 154.432 190.5)
+        (xy 153.924 190.5)
+        (xy 153.924 189.738)
+      )
+    )
+  )
+  (zone (net 0) (net_name "") (layer "F.Cu") (hatch edge 0.5)
+    (connect_pads (clearance 0))
+    (min_thickness 0.25) (filled_areas_thickness no)
+    (keepout (tracks allowed) (vias allowed) (pads allowed) (copperpour not_allowed) (footprints allowed))
+    (fill (thermal_gap 0.5) (thermal_bridge_width 0.5))
+    (polygon
+      (pts
         (xy 58.548 104.8088)
         (xy 58.548 105.4438)
@@
     )
   )
+  (zone (net 0) (net_name "") (layers "F.Cu" "Edge.Cuts") (hatch edge 0.5)
+    (connect_pads (clearance 0))
+    (min_thickness 0.25) (filled_areas_thickness no)
+    (keepout (tracks allowed) (vias allowed) (pads allowed) (copperpour not_allowed) (footprints allowed))
+    (fill (thermal_gap 0.5) (thermal_bridge_width 0.5))
+    (polygon
+      (pts
+        (xy 64.008 194.437)
+        (xy 64.008 195.453)
+        (xy 64.77 195.453)
+        (xy 64.77 194.437)
+      )
+    )
+  )
   (zone (net 2) (net_name "GNDPWR") (layer "B.Cu") (hatch edge 0.508)
     (connect_pads (clearance 0.508))
@@
       )
     )
-  )
-  (zone (net 0) (net_name "") (layer "B.Cu") (hatch edge 0.5)
-    (connect_pads (clearance 0))
-    (min_thickness 0.25) (filled_areas_thickness no)
-    (keepout (tracks allowed) (vias allowed) (pads allowed) (copperpour not_allowed) (footprints allowed))
-    (fill (thermal_gap 0.5) (thermal_bridge_width 0.5))
-    (polygon
-      (pts
-        (xy 60.072 152.0528)
-        (xy 60.072 150.2748)
-        (xy 61.469 150.2748)
-        (xy 61.469 149.7668)
-        (xy 59.564 149.7668)
-        (xy 59.564 152.0528)
-      )
-    )

Commit message: :sparkles: Update schematic
Parts:
- removed D68: SMLE13WBC8W1, LED_SMD:LED_0603_1608Metric
- removed the R2 at (58.3, 113.6)
- removed SW67: SW_Push, Button_Switch_SMD:SW_SPST_PTS645
- added TP1: ~, Connector_Pin:Pin_D1.0mm_L10.0mm, F.Cu at (69.8, 139.7)
- added TP2: ~, Connector_Pin:Pin_D1.0mm_L10.0mm, F.Cu at (69.8, 146.1)
- added TP3: ~, Connector_Pin:Pin_D1.0mm_L10.0mm, F.Cu at (342.9, 158.8)
- added TP4: ~, Connector_Pin:Pin_D1.0mm_L10.0mm, F.Cu at (342.9, 165.1)
- SW1, SW10, SW11, SW12, SW13, SW14, SW16, SW17, SW18, SW19, SW2, SW20, SW21, SW22, SW23, SW24, SW25, SW26, SW27, SW3, SW30, SW31, SW32, SW33, SW34, SW35, SW36, SW37, SW38, SW39, SW4, SW40, SW43, SW44, SW45, SW46, SW47, SW48, SW49, SW5, SW50, SW51, SW53, SW54, SW55, SW56, SW57, SW58, SW6, SW62, SW63, SW64, SW65, SW66, SW7, SW8, SW9: footprint lib:CherryMX_Choc_V2_1u -> CherryMX_Choc_V2:CherryMX_Choc_V2_1u
- SW15, SW28, SW60: footprint lib:CherryMX_Choc_V2_15u -> CherryMX_Choc_V2:CherryMX_Choc_V2_1u
- SW29, SW52: footprint lib:CherryMX_Choc_V2_175u -> CherryMX_Choc_V2:CherryMX_Choc_V2_1u
- SW41, SW42, SW59, SW61: footprint lib:CherryMX_Choc_V2_225u -> CherryMX_Choc_V2:CherryMX_Choc_V2_1u
- moved R2 248.6 mm to (331.9, 112.4)
- moved R3 248.6 mm to (329.3, 112.4)
- moved R7 248.6 mm to (336.9, 112.4)
- moved R6 248.6 mm to (334.4, 112.4)
- moved J1 248.3 mm to (331.2, 100.6)
- moved F1 234.6 mm to (319.8, 118.7)
- moved D67 234.1 mm to (319.8, 130.8)
- moved C2 228.0 mm to (317.9, 137.8)
- moved C3 228.0 mm to (317.9, 141.6)
- moved C5 228.0 mm to (317.9, 145.4)
- moved R4 225.7 mm to (324.2, 136.5)
- moved R5 225.7 mm to (321.7, 136.5)
- moved D1 20.4 mm to (345.8, 113.0)
- moved C1 15.8 mm to (193.0, 173.5), turned to 90 degrees
- moved D2 15.2 mm to (320.2, 111.3)
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- renumbered R3 to R2, R4 to R3, R5 to R4, R6 to R5, R7 to R6, R8 to R7
Connections:
- C1 pad 1: GNDPWR -> /RESET
- C1 pad 2: /RESET -> GNDPWR
- C4 pad 1: Net-(C4-Pad1) -> Net-(U1-XTAL1)
- U1 pad 17: Net-(C4-Pad1) -> Net-(U1-XTAL1)
- Y1 pad 2: Net-(C4-Pad1) -> (no net)
- Y1 pad 3: (no net) -> Net-(U1-XTAL1)
Routing:
- net +5V: track 221.5 -> 358.4 mm, vias 6 -> 10
- net /RESET: track 168.9 -> 245.7 mm, vias 6 -> 4
- net VCC: track 186.8 -> 238.3 mm, vias 5 -> 7
- net Net-(U1-XTAL1): track 0.00 -> 42.3 mm
- net Net-(C4-Pad1): track 42.3 -> 0.00 mm
- net /D0: track 342.6 -> 364.9 mm
- net /D-: track 128.8 -> 148.2 mm
- net /D+: track 128.7 -> 147.8 mm
- net /COL11: track 297.8 -> 314.9 mm, vias 1 -> 2
- net Net-(J1-D+-PadA6): track 29.7 -> 44.7 mm
- net Net-(J1-D--PadA7): track 32.3 -> 47.0 mm
- net Net-(D38-A): track 14.2 -> 3.64 mm
- net /D1: track 376.5 -> 385.3 mm, vias 4 -> 6
- net Net-(D1-A): track 15.1 -> 6.56 mm
- net GNDPWR: track 44.6 -> 38.2 mm, vias 337 -> 118
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Other:
- board text added: "5V"
- board text added: "D30"
- board text added: "GND"
- board text added: "RST"
- board text removed: "RESET"
