File: pcb/FSK-66-20-C.kicad_pcb (KiCad board)
At the start: 2 copper layers, 285 x 94.6 mm, 163 parts, among them J1 DX07S016JA3, J2 2x3_F, SW1 SW_Push, SW10 SW_Push, SW11 SW_Push, SW12 SW_Push, SW13 SW_Push, SW14 SW_Push, SW15 SW_Push, SW16 SW_Push, SW17 SW_Push, SW18 SW_Push, SW19 SW_Push, SW2 SW_Push, SW20 SW_Push, SW21 SW_Push, SW22 SW_Push, SW23 SW_Push, SW24 SW_Push, SW25 SW_Push, SW26 SW_Push, SW27 SW_Push, SW28 SW_Push, SW29 SW_Push, SW3 SW_Push, SW30 SW_Push, SW31 SW_Push, SW32 SW_Push, SW33 SW_Push, SW34 SW_Push, SW35 SW_Push, SW36 SW_Push, SW37 SW_Push, SW38 SW_Push, SW39 SW_Push, SW4 SW_Push, SW40 SW_Push, SW41 SW_Push, SW42 SW_Push, SW43 SW_Push, SW44 SW_Push, SW45 SW_Push, SW46 SW_Push, SW47 SW_Push, SW48 SW_Push, SW49 SW_Push, SW5 SW_Push, SW50 SW_Push, SW51 SW_Push, SW52 SW_Push, SW53 SW_Push, SW54 SW_Push, SW55 SW_Push, SW56 SW_Push, SW57 SW_Push, SW58 SW_Push, SW59 SW_Push, SW6 SW_Push, SW60 SW_Push, SW61 SW_Push, SW62 SW_Push, SW63 SW_Push, SW64 SW_Push, SW65 SW_Push, SW66 SW_Push, SW7 SW_Push, SW8 SW_Push, SW9 SW_Push, U1 ATmega32U4-AU, Y1 16MHz

Commit message: :sparkles: Update PCB
Parts:
- G***: footprint lib:logo_order66 -> logo:logo_order66
- TP1, TP2, TP3, TP4: footprint Connector_Pin:Pin_D1.0mm_L10.0mm -> TestPoint:TestPoint_THTPad_D1.5mm_Drill0.7mm
- moved TP1 2.54 mm to (69.8, 142.2)
- moved TP3 2.03 mm to (342.9, 160.8)
- moved TP4 1.78 mm to (342.9, 163.3)
- moved TP2 1.27 mm to (69.8, 144.8)
- moved J1 1.24 mm to (331.2, 99.4)
Routing:
- net GNDPWR: track 38.2 -> 25.4 mm, vias 118 -> 336
- net Net-(D38-A): track 3.64 -> 15.4 mm
- net +5V: track 358.4 -> 361.8 mm
- net Net-(D49-A): track 11.6 -> 14.3 mm
- net Net-(J1-D+-PadA6): track 44.7 -> 47.1 mm
- net Net-(J1-D--PadA7): track 47.0 -> 49.5 mm
- net /RESET: track 245.7 -> 243.2 mm
- net VCC: track 238.3 -> 236.6 mm, vias 7 -> 6
- net Net-(J1-CC2): track 13.4 -> 14.6 mm
- net Net-(J1-CC1): track 15.0 -> 16.2 mm
Other:
- board size 285 x 94.6 mm -> 285 x 96.1 mm

Commit message: :sparkles: Update PCB for Kailh Choc stabilizer
Parts:
- removed C8: 1u, Capacitor_SMD:C_0603_1608Metric
- added ?: , , F.Cu at (82.6, 191.1)
- added REF**: breakaway-mousebites, Keebio-Parts:breakaway-mousebites, F.Cu at (186.8, 190.9)
- added REF**: breakaway-mousebites, Keebio-Parts:breakaway-mousebites, F.Cu at (331.2, 94.5)
- added REF**: breakaway-mousebites, Keebio-Parts:breakaway-mousebites, F.Cu at (258.1, 190.9)
- added REF**: breakaway-mousebites, Keebio-Parts:breakaway-mousebites, F.Cu at (221.2, 95.2)
- added REF**: breakaway-mousebites, Keebio-Parts:breakaway-mousebites, F.Cu at (311.5, 190.9)
- added REF**: breakaway-mousebites, Keebio-Parts:breakaway-mousebites, F.Cu at (239.0, 95.2)
- added REF**: breakaway-mousebites, Keebio-Parts:breakaway-mousebites, F.Cu at (167.8, 95.2)
- added REF**: breakaway-mousebites, Keebio-Parts:breakaway-mousebites, F.Cu at (114.3, 95.2)
- added REF**: breakaway-mousebites, Keebio-Parts:breakaway-mousebites, F.Cu at (240.2, 190.9)
- added REF**: breakaway-mousebites, Keebio-Parts:breakaway-mousebites, F.Cu at (222.4, 190.9)
- added REF**: breakaway-mousebites, Keebio-Parts:breakaway-mousebites, F.Cu at (78.7, 95.2)
- added REF**: breakaway-mousebites, Keebio-Parts:breakaway-mousebites, F.Cu at (344.4, 95.2)
- added REF**: breakaway-mousebites, Keebio-Parts:breakaway-mousebites, F.Cu at (329.3, 190.9)
- added REF**: breakaway-mousebites, Keebio-Parts:breakaway-mousebites, F.Cu at (310.2, 95.2)
- added REF**: breakaway-mousebites, Keebio-Parts:breakaway-mousebites, F.Cu at (115.6, 190.9)
- added REF**: breakaway-mousebites, Keebio-Parts:breakaway-mousebites, F.Cu at (293.7, 190.9)
- added REF**: breakaway-mousebites, Keebio-Parts:breakaway-mousebites, F.Cu at (97.8, 190.9)
- added REF**: breakaway-mousebites, Keebio-Parts:breakaway-mousebites, F.Cu at (169.0, 190.9)
- added REF**: breakaway-mousebites, Keebio-Parts:breakaway-mousebites, F.Cu at (133.4, 190.9)
- added REF**: breakaway-mousebites, Keebio-Parts:breakaway-mousebites, F.Cu at (150.0, 95.2)
- added REF**: breakaway-mousebites, Keebio-Parts:breakaway-mousebites, F.Cu at (204.6, 190.9)
- added REF**: breakaway-mousebites, Keebio-Parts:breakaway-mousebites, F.Cu at (274.6, 95.2)
- added REF**: breakaway-mousebites, Keebio-Parts:breakaway-mousebites, F.Cu at (203.4, 95.2)
- added REF**: breakaway-mousebites, Keebio-Parts:breakaway-mousebites, F.Cu at (275.9, 190.9)
- added REF**: breakaway-mousebites, Keebio-Parts:breakaway-mousebites, F.Cu at (292.4, 95.2)
- added REF**: breakaway-mousebites, Keebio-Parts:breakaway-mousebites, F.Cu at (256.8, 95.2)
- added REF**: breakaway-mousebites, Keebio-Parts:breakaway-mousebites, F.Cu at (132.2, 95.2)
- added REF**: breakaway-mousebites, Keebio-Parts:breakaway-mousebites, F.Cu at (185.6, 95.2)
- added REF**: breakaway-mousebites, Keebio-Parts:breakaway-mousebites, F.Cu at (96.5, 95.2)
- added REF**: breakaway-mousebites, Keebio-Parts:breakaway-mousebites, F.Cu at (151.2, 190.9)
- added REF**: breakaway-mousebites, Keebio-Parts:breakaway-mousebites, F.Cu at (80.0, 190.9)
- C1, C3: value 1u -> 4.7u
- C2: value 10u -> 4.7u; footprint Capacitor_SMD:C_0805_2012Metric -> Capacitor_SMD:C_0603_1608Metric
- C5: value 0.1u -> 22p
- C6: value 22p -> 0.1u
- C7: value 0.1u -> 4.7u
- SW14, SW41, SW42, SW59, SW61: footprint CherryMX_Choc_V2:CherryMX_Choc_V2_1u -> kailh_choc:CherryMX_Choc_V2_225u
- TP1, TP2, TP3, TP4: footprint TestPoint:TestPoint_THTPad_D1.5mm_Drill0.7mm -> TestPoint:TestPoint_THTPad_D1.0mm_Drill0.5mm
- moved C5 133.9 mm to (186.9, 173.5)
- moved C6 44.5 mm to (211.8, 174.8), turned to 0 degrees
- moved D61 23.9 mm to (187.8, 188.0)
- moved TP3 19.2 mm to (346.7, 142.0)
- moved TP4 19.2 mm to (346.7, 144.5)
- moved Y1 13.8 mm to (181.5, 175.1), turned to 180 degrees
- moved C4 13.3 mm to (176.5, 173.5)
- moved C7 12.6 mm to (202.7, 168.1), turned to 90 degrees
- moved D41 8.63 mm to (93.9, 150.4)
- moved D59 5.57 mm to (247.4, 186.9)
- moved D42 5.10 mm to (323.6, 168.1)
- moved G*** 3.62 mm to (237.2, 176.3)
- moved G*** 2.99 mm to (239.0, 171.2)
- moved D32 1.96 mm to (269.2, 147.8)
- moved D34 1.96 mm to (231.1, 147.8)
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Connections:
- C5 pad 1: +5V -> Net-(U1-XTAL2)
- C6 pad 1: Net-(U1-XTAL2) -> Net-(U1-AREF)
- C7 pad 1: Net-(U1-AREF) -> Net-(U1-UCAP)
Routing:
- net /COL12: track 264.9 -> 297.8 mm, vias 4 -> 5
- net Net-(U1-XTAL2): track 43.2 -> 17.5 mm
- net Net-(D61-A): track 30.7 -> 5.84 mm, vias 1 -> 0
- net /RESET: track 243.2 -> 264.4 mm
- net Net-(U1-XTAL1): track 42.3 -> 26.0 mm
- net GNDPWR: track 25.4 -> 17.6 mm, vias 336 -> 301
- net Net-(D41-A): track 14.2 -> 7.36 mm
- net /COL0: track 266.9 -> 260.6 mm, vias 0 -> 1
- net /COL1: track 271.3 -> 277.6 mm
- net /D3: track 313.6 -> 319.7 mm, vias 10 -> 3
- net /D4: track 332.3 -> 338.0 mm
- net /COL4: track 187.1 -> 192.3 mm
- net VCC: track 236.6 -> 241.6 mm
- net /D1: track 385.3 -> 380.4 mm, vias 6 -> 4
- net /A0: track 204.2 -> 208.7 mm
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Other:
- board size 285 x 96.1 mm -> 285 x 107.3 mm

Commit message: :sparkles: Update PCB
Parts:
- removed the REF** at (240.2, 190.9)
- removed the REF** at (115.6, 190.9)
- removed the REF** at (293.7, 190.9)
- removed the REF** at (169.0, 190.9)
- removed the REF** at (150.0, 95.2)
- removed the REF** at (203.4, 95.2)
- removed the REF** at (256.8, 95.2)
- removed the REF** at (96.5, 95.2)
- added REF**: Fiducial_1.5mm_Mask3mm, Fiducial:Fiducial_1.5mm_Mask3mm, F.Cu at (344.2, 91.4)
- added REF**: Fiducial_1mm_Mask2mm, Fiducial:Fiducial_1mm_Mask2mm, F.Cu at (71.1, 194.3)
- added REF**: Fiducial_0.75mm_Mask1.5mm, Fiducial:Fiducial_0.75mm_Mask1.5mm, F.Cu at (337.8, 194.3)
Other:
- board size 285 x 107.3 mm -> 285 x 108.3 mm
