File: pcb/FSK-66-20-C.kicad_pcb (KiCad board)
At the start: 2 copper layers, 285 x 108.3 mm, 189 parts, among them J1 DX07S016JA3, J2 2x3_F, SW1 SW_Push, SW10 SW_Push, SW11 SW_Push, SW12 SW_Push, SW13 SW_Push, SW14 SW_Push, SW15 SW_Push, SW16 SW_Push, SW17 SW_Push, SW18 SW_Push, SW19 SW_Push, SW2 SW_Push, SW20 SW_Push, SW21 SW_Push, SW22 SW_Push, SW23 SW_Push, SW24 SW_Push, SW25 SW_Push, SW26 SW_Push, SW27 SW_Push, SW28 SW_Push, SW29 SW_Push, SW3 SW_Push, SW30 SW_Push, SW31 SW_Push, SW32 SW_Push, SW33 SW_Push, SW34 SW_Push, SW35 SW_Push, SW36 SW_Push, SW37 SW_Push, SW38 SW_Push, SW39 SW_Push, SW4 SW_Push, SW40 SW_Push, SW41 SW_Push, SW42 SW_Push, SW43 SW_Push, SW44 SW_Push, SW45 SW_Push, SW46 SW_Push, SW47 SW_Push, SW48 SW_Push, SW49 SW_Push, SW5 SW_Push, SW50 SW_Push, SW51 SW_Push, SW52 SW_Push, SW53 SW_Push, SW54 SW_Push, SW55 SW_Push, SW56 SW_Push, SW57 SW_Push, SW58 SW_Push, SW59 SW_Push, SW6 SW_Push, SW60 SW_Push, SW61 SW_Push, SW62 SW_Push, SW63 SW_Push, SW64 SW_Push, SW65 SW_Push, SW66 SW_Push, SW7 SW_Push, SW8 SW_Push, SW9 SW_Push, U1 ATmega32U4-AU, Y1 16MHz

Commit message: :sparkles: Update PCB
Parts:
- added C10: 0.1u, Capacitor_SMD:C_0402_1005Metric, F.Cu at (210.3, 183.1)
- added C11: 0.1u, Capacitor_SMD:C_0402_1005Metric, F.Cu at (211.3, 173.0)
- added C8: 0.1u, Capacitor_SMD:C_0402_1005Metric, F.Cu at (199.6, 185.4)
- added C9: 0.1u, Capacitor_SMD:C_0402_1005Metric, F.Cu at (195.3, 175.0)
- C4, C5, C6: footprint Capacitor_SMD:C_0603_1608Metric -> Capacitor_SMD:C_0402_1005Metric
- J1: value DX07S016JA3 -> USB type-C; footprint snapeda:JAE_DX07S016JA1R1500 -> Connector_USB:USB_C_Receptacle_Palconn_UTC16-G
- R1, R2, R3, R4, R5, R6, R7: footprint Resistor_SMD:R_0603_1608Metric -> Resistor_SMD:R_0402_1005Metric
- SW14, SW41, SW42, SW59, SW61: footprint kailh_choc:CherryMX_Choc_V2_225u -> CherryMX_Choc_V2:CherryMX_Choc_V2_1u
- Y1: footprint Crystal:Crystal_SMD_SeikoEpson_FA238-4Pin_3.2x2.5mm_HandSoldering -> Crystal:Crystal_SMD_SeikoEpson_FA238-4Pin_3.2x2.5mm
- moved TP1 103.9 mm to (168.9, 173.7)
- moved TP2 103.9 mm to (168.9, 176.0)
- moved G*** 32.3 mm to (268.5, 184.4)
- moved G*** 31.1 mm to (268.2, 179.3)
- moved R5 29.8 mm to (330.2, 107.9)
- moved R4 29.6 mm to (332.0, 108.0)
- moved C4 16.5 mm to (191.0, 181.4)
- moved Y1 9.79 mm to (190.8, 178.4), turned to 90 degrees
- moved D41 7.49 mm to (86.4, 150.4)
- moved D42 4.83 mm to (328.4, 168.0)
- moved C5 3.45 mm to (189.7, 175.5), turned to 180 degrees
- moved R7 2.31 mm to (334.6, 112.0)
- moved R2 2.19 mm to (329.7, 112.0)
- moved C2 1.65 mm to (319.5, 139.4)
- moved C3 1.65 mm to (319.5, 141.6)
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Connections:
- Y1 pad 1: Net-(U1-XTAL2) -> Net-(U1-XTAL1)
- Y1 pad 2: (no net) -> GNDPWR
- Y1 pad 3: Net-(U1-XTAL1) -> Net-(U1-XTAL2)
- Y1 pad 4: (no net) -> GNDPWR
Routing:
- net +5V: track 361.9 -> 269.9 mm, vias 10 -> 7
- net Net-(J1-D--PadA7): track 49.5 -> 9.02 mm
- net Net-(J1-D+-PadA6): track 47.1 -> 9.55 mm, vias 2 -> 0
- net /D+: track 145.3 -> 178.0 mm
- net /D-: track 145.3 -> 177.5 mm
- net /COL12: track 297.8 -> 270.0 mm, vias 5 -> 4
- net Net-(U1-XTAL1): track 26.0 -> 10.7 mm
- net /D4: track 338.0 -> 349.3 mm
- net GNDPWR: track 17.6 -> 27.8 mm, vias 301 -> 335
- net Net-(D41-A): track 7.36 -> 16.7 mm
- net Net-(U1-XTAL2): track 17.5 -> 9.32 mm
- net /D3: track 319.7 -> 313.2 mm
- net /D2: track 310.9 -> 317.1 mm
- net /D1: track 380.4 -> 386.2 mm
- net /COL1: track 277.6 -> 272.1 mm
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Other:
- outline, holes or cut-outs redrawn

Commit message: :sparkles: Update PCB
Routing:
- net GNDPWR: track 27.8 -> 47.0 mm, vias 335 -> 375
- net /A1: track 187.4 -> 189.7 mm
- net /A0: track 207.9 -> 209.0 mm
- net /COL1: track 272.1 -> 271.1 mm
- net /COL12: track 270.0 -> 270.9 mm
- net /D0: track 368.9 -> 368.1 mm
- net /D4: track 349.3 -> 348.5 mm
- net /A2: track 165.2 -> 164.5 mm
- net /D1: track 386.2 -> 385.6 mm
- net VCC: track 241.0 -> 240.4 mm
