File: pcb/FSK-66-20-C.kicad_sch (KiCad schematic)
At the start: 156 parts, among them J1 DX07S016JA3, J2 2x3_F, SW1 SW_Push, SW10 SW_Push, SW11 SW_Push, SW12 SW_Push, SW13 SW_Push, SW14 SW_Push, SW15 SW_Push, SW16 SW_Push, SW17 SW_Push, SW18 SW_Push, SW19 SW_Push, SW2 SW_Push, SW20 SW_Push, SW21 SW_Push, SW22 SW_Push, SW23 SW_Push, SW24 SW_Push, SW25 SW_Push, SW26 SW_Push, SW27 SW_Push, SW28 SW_Push, SW29 SW_Push, SW3 SW_Push, SW30 SW_Push, SW31 SW_Push, SW32 SW_Push, SW33 SW_Push, SW34 SW_Push, SW35 SW_Push, SW36 SW_Push, SW37 SW_Push, SW38 SW_Push, SW39 SW_Push, SW4 SW_Push, SW40 SW_Push, SW41 SW_Push, SW42 SW_Push, SW43 SW_Push, SW44 SW_Push, SW45 SW_Push, SW46 SW_Push, SW47 SW_Push, SW48 SW_Push, SW49 SW_Push, SW5 SW_Push, SW50 SW_Push, SW51 SW_Push, SW52 SW_Push, SW53 SW_Push, SW54 SW_Push, SW55 SW_Push, SW56 SW_Push, SW57 SW_Push, SW58 SW_Push, SW59 SW_Push, SW6 SW_Push, SW60 SW_Push, SW61 SW_Push, SW62 SW_Push, SW63 SW_Push, SW64 SW_Push, SW65 SW_Push, SW66 SW_Push, SW67 SW_Push, SW7 SW_Push, SW8 SW_Push, SW9 SW_Push, U1 ATmega32U4-AU, Y1 16MHz

Commit message: :sparkles: Update schematic
Parts:
- removed D68: SMLE13WBC8W1, LED_SMD:LED_0603_1608Metric, symbol Device:LED_Small
- removed R2: 10k, Resistor_SMD:R_0603_1608Metric, symbol Device:R_US
- added TP1, TP2, TP3, TP4: ~, symbol Connector:TestPoint
Connections:
- net +5V: now also TP1.1
- net GNDPWR: now also TP2.1, TP4.1
- net RESET: now also TP3.1
Other:
- title: 66 Keys full size keyboard -> 66 Keys keyboard

Commit message: :sparkles: Update schematic
Parts:
- removed SW67: SW_Push, Button_Switch_SMD:SW_SPST_PTS645, symbol Switch:SW_Push
- TP1: renamed from TP3; footprint (none) -> Connector_Pin:Pin_D1.0mm_L10.0mm
- TP2: renamed from TP4; footprint (none) -> Connector_Pin:Pin_D1.0mm_L10.0mm
- TP3: renamed from TP1; footprint (none) -> Connector_Pin:Pin_D1.0mm_L10.0mm
- TP4: renamed from TP2; footprint (none) -> Connector_Pin:Pin_D1.0mm_L10.0mm
- renumbered C2 to C1, C3 to C2, C5 to C3, C6 to C5, C1 to C6, D56 to D10, D67 to D11, D3 to D12, D17 to D13, D31 to D14, D44 to D15, D57 to D16, D4 to D17, D32 to D19, D15 to D2, D45 to D20, D58 to D21, D5 to D22, D19 to D23, D33 to D24, D46 to D25, D59 to D26, D6 to D27, D20 to D28, D34 to D29, D29 to D3, D47 to D30, D60 to D31, D7 to D32, D21 to D33, D35 to D34, D48 to D35, D61 to D36, D8 to D37, D22 to D38, D36 to D39, D42 to D4, D49 to D40, D62 to D41, D9 to D42, D23 to D43, D37 to D44, D50 to D45, D63 to D46, D10 to D47, D24 to D48, D38 to D49, D55 to D5, D51 to D50, D64 to D51, D11 to D52, D25 to D53, D39 to D54, D52 to D55, D65 to D56, D12 to D57, D26 to D58, D40 to D59, D2 to D6, D53 to D60, D66 to D61, D13 to D62, D27 to D63, D41 to D64, D54 to D65, D14 to D66, D28 to D67, D16 to D7, D30 to D8, D43 to D9, R5 to R1, R6 to R2, R7 to R5, R8 to R6, R1 to R7, SW56 to SW10, SW3 to SW11, SW17 to SW12, SW31 to SW13, SW44 to SW14, SW57 to SW15, SW4 to SW16, SW18 to SW17, SW32 to SW18, SW45 to SW19, SW15 to SW2, SW58 to SW20, SW5 to SW21, SW19 to SW22, SW33 to SW23, SW46 to SW24, SW59 to SW25, SW6 to SW26, SW20 to SW27, SW34 to SW28, SW47 to SW29, SW29 to SW3, SW60 to SW30, SW7 to SW32, SW21 to SW33, SW35 to SW34, SW48 to SW35, SW61 to SW36, SW8 to SW37, SW22 to SW38, SW36 to SW39, SW42 to SW4, SW49 to SW40, SW62 to SW41, SW9 to SW42, SW23 to SW43, SW37 to SW44, SW50 to SW45, SW63 to SW46, SW10 to SW47, SW24 to SW48, SW38 to SW49, SW55 to SW5, SW51 to SW50, SW64 to SW51, SW11 to SW52, SW25 to SW53, SW39 to SW54, SW52 to SW55, SW65 to SW56, SW12 to SW57, SW26 to SW58, SW40 to SW59, SW2 to SW6, SW53 to SW60, SW66 to SW61, SW13 to SW62, SW27 to SW63, SW41 to SW64, SW54 to SW65, SW14 to SW66, SW28 to SW67, SW16 to SW7, SW30 to SW8, SW43 to SW9
Connections:
- net GNDPWR: now also C6.2; no longer C6.1
- net RESET: now also C6.1; no longer C6.2
Other:
- moved on the sheet: C6, R7

Commit message: :sparkles: Update schematic
Parts:
- SW1: footprint keyboard_toms:CherryMX_Choc_V2_1u -> CherryMX_Choc_V2:CherryMX_Choc_V2_1u
- SW10: renamed from SW47; footprint keyboard_toms:CherryMX_Choc_V2_1u -> CherryMX_Choc_V2:CherryMX_Choc_V2_1u
- SW11: renamed from SW52; footprint keyboard_toms:CherryMX_Choc_V2_1u -> CherryMX_Choc_V2:CherryMX_Choc_V2_1u
- SW12: renamed from SW57; footprint keyboard_toms:CherryMX_Choc_V2_1u -> CherryMX_Choc_V2:CherryMX_Choc_V2_1u
- SW13: renamed from SW62; footprint keyboard_toms:CherryMX_Choc_V2_1u -> CherryMX_Choc_V2:CherryMX_Choc_V2_1u
- SW14: renamed from SW66; footprint keyboard_toms:CherryMX_Choc_V2_1u -> CherryMX_Choc_V2:CherryMX_Choc_V2_1u
- SW15: renamed from SW2; footprint keyboard_toms:CherryMX_Choc_V2_1u -> CherryMX_Choc_V2:CherryMX_Choc_V2_1u
- SW16: renamed from SW7; footprint keyboard_toms:CherryMX_Choc_V2_1u -> CherryMX_Choc_V2:CherryMX_Choc_V2_1u
- SW17: renamed from SW12; footprint keyboard_toms:CherryMX_Choc_V2_1u -> CherryMX_Choc_V2:CherryMX_Choc_V2_1u
- SW18: renamed from SW17; footprint keyboard_toms:CherryMX_Choc_V2_1u -> CherryMX_Choc_V2:CherryMX_Choc_V2_1u
- SW19: renamed from SW22; footprint keyboard_toms:CherryMX_Choc_V2_1u -> CherryMX_Choc_V2:CherryMX_Choc_V2_1u
- SW2: renamed from SW6; footprint keyboard_toms:CherryMX_Choc_V2_1u -> CherryMX_Choc_V2:CherryMX_Choc_V2_1u
- SW20: renamed from SW27; footprint keyboard_toms:CherryMX_Choc_V2_1u -> CherryMX_Choc_V2:CherryMX_Choc_V2_1u
- SW21: renamed from SW33; footprint keyboard_toms:CherryMX_Choc_V2_1u -> CherryMX_Choc_V2:CherryMX_Choc_V2_1u
- SW22: renamed from SW38; footprint keyboard_toms:CherryMX_Choc_V2_1u -> CherryMX_Choc_V2:CherryMX_Choc_V2_1u
- SW23: renamed from SW43; footprint keyboard_toms:CherryMX_Choc_V2_1u -> CherryMX_Choc_V2:CherryMX_Choc_V2_1u
- SW24: renamed from SW48; footprint keyboard_toms:CherryMX_Choc_V2_1u -> CherryMX_Choc_V2:CherryMX_Choc_V2_1u
- SW25: renamed from SW53; footprint keyboard_toms:CherryMX_Choc_V2_1u -> CherryMX_Choc_V2:CherryMX_Choc_V2_1u
- SW26: renamed from SW58; footprint keyboard_toms:CherryMX_Choc_V2_1u -> CherryMX_Choc_V2:CherryMX_Choc_V2_1u
- SW27: renamed from SW63; footprint keyboard_toms:CherryMX_Choc_V2_1u -> CherryMX_Choc_V2:CherryMX_Choc_V2_1u
- SW28: renamed from SW67; footprint keyboard_toms:CherryMX_Choc_V2_1u -> CherryMX_Choc_V2:CherryMX_Choc_V2_1u
- SW29: renamed from SW3; footprint keyboard_toms:CherryMX_Choc_V2_1u -> CherryMX_Choc_V2:CherryMX_Choc_V2_1u
- SW3: renamed from SW11; footprint keyboard_toms:CherryMX_Choc_V2_1u -> CherryMX_Choc_V2:CherryMX_Choc_V2_1u
- SW30: renamed from SW8; footprint keyboard_toms:CherryMX_Choc_V2_1u -> CherryMX_Choc_V2:CherryMX_Choc_V2_1u
- SW31: renamed from SW13; footprint keyboard_toms:CherryMX_Choc_V2_1u -> CherryMX_Choc_V2:CherryMX_Choc_V2_1u
- SW32: renamed from SW18; footprint keyboard_toms:CherryMX_Choc_V2_1u -> CherryMX_Choc_V2:CherryMX_Choc_V2_1u
- SW33: renamed from SW23; footprint keyboard_toms:CherryMX_Choc_V2_1u -> CherryMX_Choc_V2:CherryMX_Choc_V2_1u
- SW34: renamed from SW28; footprint keyboard_toms:CherryMX_Choc_V2_1u -> CherryMX_Choc_V2:CherryMX_Choc_V2_1u
- SW35: renamed from SW34; footprint keyboard_toms:CherryMX_Choc_V2_1u -> CherryMX_Choc_V2:CherryMX_Choc_V2_1u
- SW36: renamed from SW39; footprint keyboard_toms:CherryMX_Choc_V2_1u -> CherryMX_Choc_V2:CherryMX_Choc_V2_1u
- SW37: renamed from SW44; footprint keyboard_toms:CherryMX_Choc_V2_1u -> CherryMX_Choc_V2:CherryMX_Choc_V2_1u
- SW38: renamed from SW49; footprint keyboard_toms:CherryMX_Choc_V2_1u -> CherryMX_Choc_V2:CherryMX_Choc_V2_1u
- SW39: renamed from SW54; footprint keyboard_toms:CherryMX_Choc_V2_1u -> CherryMX_Choc_V2:CherryMX_Choc_V2_1u
- SW4: renamed from SW16; footprint keyboard_toms:CherryMX_Choc_V2_1u -> CherryMX_Choc_V2:CherryMX_Choc_V2_1u
- SW40: renamed from SW59; footprint keyboard_toms:CherryMX_Choc_V2_1u -> CherryMX_Choc_V2:CherryMX_Choc_V2_1u
- SW41: renamed from SW64; footprint keyboard_toms:CherryMX_Choc_V2_1u -> CherryMX_Choc_V2:CherryMX_Choc_V2_1u
- SW42: renamed from SW4; footprint keyboard_toms:CherryMX_Choc_V2_1u -> CherryMX_Choc_V2:CherryMX_Choc_V2_1u
- SW43: renamed from SW9; footprint keyboard_toms:CherryMX_Choc_V2_1u -> CherryMX_Choc_V2:CherryMX_Choc_V2_1u
- SW44: renamed from SW14; footprint keyboard_toms:CherryMX_Choc_V2_1u -> CherryMX_Choc_V2:CherryMX_Choc_V2_1u
- SW45: renamed from SW19; footprint keyboard_toms:CherryMX_Choc_V2_1u -> CherryMX_Choc_V2:CherryMX_Choc_V2_1u
- SW46: renamed from SW24; footprint keyboard_toms:CherryMX_Choc_V2_1u -> CherryMX_Choc_V2:CherryMX_Choc_V2_1u
- SW47: renamed from SW29; footprint keyboard_toms:CherryMX_Choc_V2_1u -> CherryMX_Choc_V2:CherryMX_Choc_V2_1u
- SW48: renamed from SW35; footprint keyboard_toms:CherryMX_Choc_V2_1u -> CherryMX_Choc_V2:CherryMX_Choc_V2_1u
- SW49: renamed from SW40; footprint keyboard_toms:CherryMX_Choc_V2_1u -> CherryMX_Choc_V2:CherryMX_Choc_V2_1u
- SW5: renamed from SW21; footprint keyboard_toms:CherryMX_Choc_V2_1u -> CherryMX_Choc_V2:CherryMX_Choc_V2_1u
- SW50: renamed from SW45; footprint keyboard_toms:CherryMX_Choc_V2_1u -> CherryMX_Choc_V2:CherryMX_Choc_V2_1u
- SW51: renamed from SW50; footprint keyboard_toms:CherryMX_Choc_V2_1u -> CherryMX_Choc_V2:CherryMX_Choc_V2_1u
- SW52: renamed from SW55; footprint keyboard_toms:CherryMX_Choc_V2_1u -> CherryMX_Choc_V2:CherryMX_Choc_V2_1u
- SW53: renamed from SW60; footprint keyboard_toms:CherryMX_Choc_V2_1u -> CherryMX_Choc_V2:CherryMX_Choc_V2_1u
- SW54: renamed from SW65; footprint keyboard_toms:CherryMX_Choc_V2_1u -> CherryMX_Choc_V2:CherryMX_Choc_V2_1u
- SW55: renamed from SW5; footprint keyboard_toms:CherryMX_Choc_V2_1u -> CherryMX_Choc_V2:CherryMX_Choc_V2_1u
- SW56: renamed from SW10; footprint keyboard_toms:CherryMX_Choc_V2_1u -> CherryMX_Choc_V2:CherryMX_Choc_V2_1u
- SW57: renamed from SW15; footprint keyboard_toms:CherryMX_Choc_V2_1u -> CherryMX_Choc_V2:CherryMX_Choc_V2_1u
- SW58: renamed from SW20; footprint keyboard_toms:CherryMX_Choc_V2_1u -> CherryMX_Choc_V2:CherryMX_Choc_V2_1u
- SW59: renamed from SW25; footprint keyboard_toms:CherryMX_Choc_V2_1u -> CherryMX_Choc_V2:CherryMX_Choc_V2_1u
- SW6: renamed from SW26; footprint keyboard_toms:CherryMX_Choc_V2_1u -> CherryMX_Choc_V2:CherryMX_Choc_V2_1u
- SW60: renamed from SW30; footprint keyboard_toms:CherryMX_Choc_V2_1u -> CherryMX_Choc_V2:CherryMX_Choc_V2_1u
- SW61: renamed from SW36; footprint keyboard_toms:CherryMX_Choc_V2_1u -> CherryMX_Choc_V2:CherryMX_Choc_V2_1u
- SW62: renamed from SW41; footprint keyboard_toms:CherryMX_Choc_V2_1u -> CherryMX_Choc_V2:CherryMX_Choc_V2_1u
- SW63: renamed from SW46; footprint keyboard_toms:CherryMX_Choc_V2_1u -> CherryMX_Choc_V2:CherryMX_Choc_V2_1u
- SW64: renamed from SW51; footprint keyboard_toms:CherryMX_Choc_V2_1u -> CherryMX_Choc_V2:CherryMX_Choc_V2_1u
- SW65: renamed from SW56; footprint keyboard_toms:CherryMX_Choc_V2_1u -> CherryMX_Choc_V2:CherryMX_Choc_V2_1u
- SW66: renamed from SW61; footprint keyboard_toms:CherryMX_Choc_V2_1u -> CherryMX_Choc_V2:CherryMX_Choc_V2_1u
- SW7: renamed from SW32; footprint keyboard_toms:CherryMX_Choc_V2_1u -> CherryMX_Choc_V2:CherryMX_Choc_V2_1u
- SW8: renamed from SW37; footprint keyboard_toms:CherryMX_Choc_V2_1u -> CherryMX_Choc_V2:CherryMX_Choc_V2_1u
- SW9: renamed from SW42; footprint keyboard_toms:CherryMX_Choc_V2_1u -> CherryMX_Choc_V2:CherryMX_Choc_V2_1u
- renumbered C6 to C1, C1 to C2, C2 to C3, C3 to C5, C5 to C6, D47 to D10, D52 to D11, D57 to D12, D62 to D13, D66 to D14, D2 to D15, D7 to D16, D13 to D17, D23 to D19, D6 to D2, D28 to D20, D33 to D21, D38 to D22, D43 to D23, D48 to D24, D53 to D25, D58 to D26, D63 to D27, D67 to D28, D3 to D29, D12 to D3, D8 to D30, D14 to D31, D19 to D32, D24 to D33, D29 to D34, D34 to D35, D39 to D36, D44 to D37, D49 to D38, D54 to D39, D17 to D4, D59 to D40, D64 to D41, D4 to D42, D9 to D43, D15 to D44, D20 to D45, D25 to D46, D30 to D47, D35 to D48, D40 to D49, D22 to D5, D45 to D50, D50 to D51, D55 to D52, D60 to D53, D65 to D54, D5 to D55, D10 to D56, D16 to D57, D21 to D58, D26 to D59, D27 to D6, D31 to D60, D36 to D61, D41 to D62, D46 to D63, D51 to D64, D56 to D65, D61 to D66, D11 to D67, D32 to D7, D37 to D8, D42 to D9, R7 to R1, R3 to R2, R4 to R3, R1 to R4, R2 to R5, R5 to R6, R6 to R7, TP3 to TP1, TP4 to TP2, TP1 to TP3, TP2 to TP4

Commit message: :sparkles: Update PCB
Parts:
- TP1, TP2, TP3, TP4: footprint Connector_Pin:Pin_D1.0mm_L10.0mm -> TestPoint:TestPoint_THTPad_D1.0mm_Drill0.5mm
Changed lines of the file:
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@@
 			)
 		)
-		(property "Footprint" "Connector_Pin:Pin_D1.0mm_L10.0mm"
+		(property "Footprint" "TestPoint:TestPoint_THTPad_D1.0mm_Drill0.5mm"
 			(at 109.22 242.57 0)
 			(effects
@@
 			)
 		)
-		(property "Footprint" "Connector_Pin:Pin_D1.0mm_L10.0mm"
+		(property "Footprint" "TestPoint:TestPoint_THTPad_D1.0mm_Drill0.5mm"
 			(at 144.78 171.45 0)
 			(effects
@@
 			)
 		)
-		(property "Footprint" "Connector_Pin:Pin_D1.0mm_L10.0mm"
+		(property "Footprint" "TestPoint:TestPoint_THTPad_D1.0mm_Drill0.5mm"
 			(at 154.94 201.93 0)
 			(effects
@@
 			)
 		)
-		(property "Footprint" "Connector_Pin:Pin_D1.0mm_L10.0mm"
+		(property "Footprint" "TestPoint:TestPoint_THTPad_D1.0mm_Drill0.5mm"
 			(at 99.06 231.14 0)
 			(effects

Commit message: :sparkles: Update schematic
Parts:
- removed C5: 0.1u, Capacitor_SMD:C_0603_1608Metric, symbol Device:C
- C1, C3: value 1u -> 4.7u
- C2: value 10u -> 4.7u; footprint Capacitor_SMD:C_0805_2012Metric -> Capacitor_SMD:C_0603_1608Metric
- C7: renamed from C8; value 1u -> 4.7u
- renumbered C6 to C5, C7 to C6
Other:
- moved on the sheet: C7, TP1, TP2

Commit message: :sparkles: Update schematic
Parts:
- added C10, C11, C8, C9: 0.1u, Capacitor_SMD:C_0402_1005Metric, symbol Device:C
- C4, C5, C6: footprint Capacitor_SMD:C_0603_1608Metric -> Capacitor_SMD:C_0402_1005Metric
- J1: value DX07S016JA3 -> USB type-C; footprint snapeda:JAE_DX07S016JA1R1500 -> Connector_USB:USB_C_Receptacle_Palconn_UTC16-G
- R1, R2, R3, R4, R5, R6, R7: footprint Resistor_SMD:R_0603_1608Metric -> Resistor_SMD:R_0402_1005Metric
- Y1: footprint Crystal:Crystal_SMD_SeikoEpson_FA238-4Pin_3.2x2.5mm_HandSoldering -> Crystal:Crystal_SMD_SeikoEpson_FA238-4Pin_3.2x2.5mm; symbol Device:Crystal_Small -> Device:Crystal_GND24
Connections:
- net +5V: now also C10.1, C11.1, C8.1, C9.1
- net GNDPWR: now also Y1.2, Y1.4, C10.2, C11.2, C8.2, C9.2
- net at C5.1, U1.16 (XTAL2): now also Y1.3; no longer Y1.1
- net at C4.1, U1.17 (XTAL1): now also Y1.1; no longer Y1.2
Other:
- moved on the sheet: C4, C5
