File: plates/order66_switch_plate.kicad_pcb (KiCad board)
At the start: 2 copper layers, 285 x 94.6 mm, 65 parts, among them SW1 SW_Push, SW10 SW_Push, SW11 SW_Push, SW12 SW_Push, SW13 SW_Push, SW15 SW_Push, SW16 SW_Push, SW17 SW_Push, SW18 SW_Push, SW19 SW_Push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

Commit message: :sparkles: Update switch plate for Kailh Choc stabilizer
Parts:
- REF** (x5): footprint BrownSugar_KBD:Stabilizer_MX_Plate_Mount_2U -> kailh_choc:Kailh_Choc_2u_Stabilizer_Cutout
- turned REF** to 180 degrees (x4)
Other:
- outline, holes or cut-outs redrawn
