File: plates/middle/order66_middle_plate.kicad_pcb (KiCad board)
At the start: 2 copper layers, 285 x 94.6 mm, 60 parts, among them SW1 SW_Push, SW10 SW_Push, SW11 SW_Push, SW12 SW_Push, SW13 SW_Push, SW15 SW_Push, SW16 SW_Push, SW17 SW_Push, SW18 SW_Push, SW19 SW_Push, SW2 SW_Push, SW20 SW_Push, SW21 SW_Push, SW22 SW_Push, SW23 SW_Push, SW24 SW_Push, SW25 SW_Push, SW26 SW_Push, SW27 SW_Push, SW28 SW_Push, SW29 SW_Push, SW3 SW_Push, SW30 SW_Push, SW31 SW_Push, SW32 SW_Push, SW33 SW_Push, SW36 SW_Push, SW37 SW_Push, SW38 SW_Push, SW39 SW_Push, SW4 SW_Push, SW40 SW_Push, SW43 SW_Push, SW44 SW_Push, SW45 SW_Push, SW46 SW_Push, SW47 SW_Push, SW48 SW_Push, SW49 SW_Push, SW5 SW_Push, SW50 SW_Push, SW51 SW_Push, SW52 SW_Push, SW53 SW_Push, SW54 SW_Push, SW55 SW_Push, SW56 SW_Push, SW57 SW_Push, SW58 SW_Push, SW6 SW_Push, SW60 SW_Push, SW63 SW_Push, SW64 SW_Push, SW65 SW_Push, SW66 SW_Push, SW7 SW_Push, SW8 SW_Push, SW9 SW_Push

Commit message: :sparkles: Update middle plate
Parts:
- added REF**: Stabilizer 2U, plate:CherryMX_Choc_V2_1u, F.Cu at (328.7, 162.1)
- added REF**: Stabilizer 2U, plate:CherryMX_Choc_V2_1u, F.Cu at (86.5, 143.1)
- added REF**: Stabilizer 2U, plate:CherryMX_Choc_V2_1u, F.Cu at (252.7, 181.1)
- added REF**: Stabilizer 2U, plate:CherryMX_Choc_V2_1u, F.Cu at (83.1, 105.1)
- added REF**: Stabilizer 2U, plate:CherryMX_Choc_V2_1u, F.Cu at (181.4, 181.1)
Other:
- outline, holes or cut-outs redrawn
