File: plates/top/order66_switch_plate.kicad_pcb (KiCad board)
At the start: 2 copper layers, 285 x 94.6 mm, 65 parts, among them SW1 SW_Push, SW10 SW_Push, SW11 SW_Push, SW12 SW_Push, SW13 SW_Push, SW15 SW_Push, SW16 SW_Push, SW17 SW_Push, SW18 SW_Push, SW19 SW_Push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

Commit message: :sparkles: Update top plate
Parts:
- REF** (x5): footprint kailh_choc:Kailh_Choc_2u_Stabilizer_Cutout -> plate:CherryMX_Choc_V2_1u
Other:
- outline, holes or cut-outs redrawn
- board text added: "GND"
- board text added: "RST"
